Commit message: Demo scene working, somewhat

File: src/demo_world/urdf/conveyor.urdf (robot description, URDF)
Before this commit: robot liukuhihna_gazebo, 3 links, 2 joints
Links:
- link belt_visual: geometry collision box size=0.463 1.2 0.73; visual mesh filename=package://demo_world/meshes/conveyor_belt.stl

Commit message: CV2 testing

File: src/demo_world/urdf/conveyor.urdf (robot description, URDF)
Before this commit: robot liukuhihna_gazebo, 3 links, 2 joints
Links:
- link belt_visual: geometry collision mesh filename=package://demo_world/meshes/conveyor_simple.stl; visual mesh filename=package://demo_world/meshes/conveyor_belt.stl

File: src/demo_world/urdf/samk_2f_85_depth.urdf.xacro (robot description, xacro)
@@ -7,5 +7,10 @@
   <xacro:robotiq_arg2f_85 prefix="robotiq_"/>
   <!-- Intel RealSense D435 -->
-  <xacro:include filename="$(find demo_world)/urdf/d435_camera.urdf.xacro" />
+  <xacro:arg name="use_nominal_extrinsics" default="true"/>
+  <xacro:arg name="add_plug" default="false" />
+  <xacro:include filename="$(find demo_world)/urdf/_d435.urdf.xacro" />
+  <xacro:sensor_d435 parent="elfin_end_link" use_nominal_extrinsics="$(arg use_nominal_extrinsics)">
+    <origin xyz="-0.045 0 0.02" rpy="0 -${pi/2} 0"/>
+  </xacro:sensor_d435>
   <!-- TOOL CONNECTOR -->
   <joint name="tool_connector" type="fixed">
@@ -26,6 +31,6 @@
     <kp>1e+13</kp>
     <kd>1</kd>
-    <!--<max_vel>0.01</max_vel>
-      <min_depth>0</min_depth>-->
+    <!-- <max_vel>0.01</max_vel> -->
+    <!-- <min_depth>0</min_depth> -->
     <sensor name="color" type="camera">
       <camera name="realsense">
@@ -58,8 +63,8 @@
           <format>L_INT8</format>
         </image>
-        <clip>
+        <!-- <clip>
           <near>0.1</near>
           <far>100</far>
-        </clip>
+        </clip> -->
         <noise>
           <type>gaussian</type>
@@ -80,8 +85,8 @@
           <format>L_INT8</format>
         </image>
-        <clip>
+        <!-- <clip>
           <near>0.1</near>
           <far>100</far>
-        </clip>
+        </clip> -->
         <noise>
           <type>gaussian</type>
@@ -101,13 +106,13 @@
           <height>720</height>
         </image>
-        <clip>
+        <!-- <clip>
           <near>0.1</near>
           <far>100</far>
-        </clip>
-        <noise>
+        </clip> -->
+        <!-- <noise>
           <type>gaussian</type>
           <mean>0.0</mean>
           <stddev>0.100</stddev>
-        </noise>
+        </noise> -->
       </camera>
       <always_on>1</always_on>
@@ -137,5 +142,5 @@
       <pointCloud>true</pointCloud>
       <pointCloudTopicName>depth/points</pointCloudTopicName>
-      <pointCloudCutoff>0.5</pointCloudCutoff>
+      <pointCloudCutoff>0.2</pointCloudCutoff>
     </plugin>
   </gazebo>
